File: starbie/starbie.kicad_sch (KiCad schematic)
At the start: 4 parts, among them SW1 SW_Push, SW2 SW_Push, U1 DHT11

Commit message: added the MPU6050 and OLED
Parts:
- added J1: Conn_01x04_Pin, symbol Connector:Conn_01x04_Pin
- added U2: XIAO-ESP32-C3-SMD, Seeed_Studio_XIAO_Series:XIAO-ESP32-C3-SMD, symbol Seeed_Studio_XIAO_Series:XIAO-ESP32-C3-SMD
Connections:
- net +3.3V: now also R1.1, U2.12 (3V3_OUT)
- net GND: now also U2.13 (GND), U2.18 (GND)
- no-connect marks 0 -> 18
