File: starbie/starbie.kicad_pcb (KiCad board)
At the start: 2 copper layers, 7 parts, among them J1 Conn_01x04_Pin, J2 Conn_01x08_Pin, SW1 SW_Push, SW2 SW_Push, U1 DHT11, U2 XIAO-ESP32-C3-SMD

Commit message: finshed pcb routing in odays session
Parts:
- moved U2 108.6 mm to (247.2, 101.9)
- moved R1 107.0 mm to (220.2, 82.5)
- moved SW2 95.3 mm to (207.3, 125.3)
- moved J2 95.0 mm to (238.5, 117.3)
- moved J1 85.2 mm to (223.0, 92.5)
- moved SW1 81.5 mm to (199.5, 93.4)
- moved U1 65.7 mm to (220.0, 87.0), turned to 90 degrees
Routing:
- net GND: track 0.00 -> 138.3 mm
- net +3.3V: track 0.00 -> 57.7 mm
Other:
- board outline added: 103.7 x 88.1 mm
