File: starbie/starbie.kicad_pcb (KiCad board)
At the start: 2 copper layers, 103.7 x 88.1 mm, 7 parts, among them J1 Conn_01x04_Pin, J2 Conn_01x08_Pin, SW1 SW_Push, SW2 SW_Push, U1 DHT11, U2 XIAO-ESP32-C3-SMD

Commit message: added the logo to pcb
Parts:
- added G***: LOGO, logo:logo, F.Cu at (225.5, 74.5)
