File: starbie/_restore_backup_2026-10-07T09-47-09-069/starbie.kicad_sch (KiCad schematic)
At the start: 7 parts, among them J1 Conn_01x04_Pin, J2 Conn_01x08_Pin, SW1 SW_Push, SW2 SW_Push, U1 DHT11, U2 XIAO-ESP32-C3-SMD

Commit message: pushing progress to save it
Parts:
- removed J2: Conn_01x08_Pin, Connector_PinHeader_2.54mm:PinHeader_1x08_P2.54mm_Vertical, symbol Connector:Conn_01x08_Pin
- J1: footprint Imported Parts:Display_128x64_096_I2C -> (none)
- R1: footprint Resistor_THT:R_Axial_DIN0204_L3.6mm_D1.6mm_P7.62mm_Horizontal -> (none)
- SW1, SW2: footprint Button_Switch_Keyboard:SW_Cherry_MX_1.00u_PCB -> Button_Switch_THT:SW_NKK_GW12LJP
- U2: footprint Imported Parts:XIAO-ESP32-C6-DIP -> Seeed_Studio_XIAO_Series:XIAO-ESP32-C3-SMD
Connections:
- net +3.3V: no longer J1.2 (Pin_2)
- net GND: no longer J1.1 (Pin_1)
- no-connect marks 22 -> 18
